Commit message: feat: Add controller manager and depth camera

File: description/robot.urdf.xacro (robot description, xacro)
@@ -2,6 +2,13 @@
 <robot xmlns:xacro="http://www.ros.org/wiki/xacro"  name="robot">
     <xacro:include filename="robot_core.xacro" />
-    <xacro:include filename="gazebo_control.xacro"/>
+    <xacro:arg name="use_ros2_control" default="true"/>
+    <xacro:if value="$(arg use_ros2_control)">
+        <xacro:include filename="ros2_control.xacro" />
+    </xacro:if>
+    <xacro:unless value="$(arg use_ros2_control)">
+        <xacro:include filename="gazebo_control.xacro" />
+    </xacro:unless>
     <xacro:include filename="lidar.xacro"/>
     <xacro:include filename="camera.xacro"/>
+    <!-- <xacro:include filename="depth_camera.xacro"/> -->
 </robot>

File: description/robot_core.xacro (robot description, xacro)
@@ -59,5 +59,5 @@
     <collision>
       <geometry>
-        <cylinder radius="0.05" length="0.04"/>
+        <sphere radius="0.05"/>
       </geometry>
     </collision>
@@ -84,5 +84,5 @@
     <collision>
       <geometry>
-        <cylinder radius="0.05" length="0.04"/>
+        <sphere radius="0.05"/>
       </geometry>
     </collision>
