Commit message: feat: add gazebo simulation and control

File: description/robot_core.xacro (robot description, xacro)
@@ -1,4 +1,4 @@
 <?xml version="1.0"?>
-<robot xmlns:xacro="http://www.ros.org/wiki/xacro" >
+<robot xmlns:xacro="http://www.ros.org/wiki/xacro">
   <xacro:include filename="inertial_macros.xacro"/>
   <material name="white">
@@ -35,8 +35,11 @@
       </geometry>
     </collision>
-    <xacro:inertial_box mass="0.5" x="0.3" y="0.3" z="-.15">
+    <xacro:inertial_box mass="0.5" x="0.3" y="0.3" z="0.15">
       <origin xyz="0.15 0 0.075" rpy="0 0 0"/>
     </xacro:inertial_box>
   </link>
+  <gazebo reference="chassis">
+    <material>Gazebo/White</material>
+  </gazebo>
   <joint name="left_wheel_joint" type="continuous">
     <parent link="base_link"/>
@@ -57,8 +60,11 @@
       </geometry>
     </collision>
-    <xacro:inertial_cylinder mass="0.1" radius="0.05" length="0.04">
+    <xacro:inertial_cylinder mass="0.1" length="0.04" radius="0.05">
       <origin xyz="0 0 0" rpy="0 0 0"/>
     </xacro:inertial_cylinder>
   </link>
+  <gazebo reference="left_wheel">
+    <material>Gazebo/Blue</material>
+  </gazebo>
   <joint name="right_wheel_joint" type="continuous">
     <parent link="base_link"/>
@@ -79,8 +85,11 @@
       </geometry>
     </collision>
-    <xacro:inertial_cylinder mass="0.1" radius="0.05" length="0.04">
+    <xacro:inertial_cylinder mass="0.1" length="0.04" radius="0.05">
       <origin xyz="0 0 0" rpy="0 0 0"/>
     </xacro:inertial_cylinder>
   </link>
+  <gazebo reference="right_wheel">
+    <material>Gazebo/Blue</material>
+  </gazebo>
   <joint name="caster_wheel_joint" type="fixed">
     <parent link="chassis"/>
@@ -104,3 +113,8 @@
     </xacro:inertial_sphere>
   </link>
+  <gazebo reference="caster_wheel">
+    <material>Gazebo/Black</material>
+    <mu1 value="0.001"/>
+    <mu2 value="0.001"/>
+  </gazebo>
 </robot>

Commit message: feat: add lidar scanner

File: description/robot_core.xacro (robot description, xacro)
@@ -14,6 +14,8 @@
     <color rgba="0 0 0 1"/>
   </material>
-  <link name="base_link">
-  </link>
+  <material name="red">
+    <color rgba="1 0 0 1"/>
+  </material>
+  <link name="base_link"></link>
   <joint name="chassis_joint" type="fixed">
     <parent link="base_link"/>

Commit message: feat: Add slam

File: description/robot_core.xacro (robot description, xacro)
@@ -18,4 +18,10 @@
   </material>
   <link name="base_link"></link>
+  <joint name="base_footprint_joint" type="fixed">
+    <parent link="base_link"/>
+    <child link="base_footprint"/>
+    <origin xyz="0 0 0" rpy="0 0 0"/>
+  </joint>
+  <link name="base_footprint"></link>
   <joint name="chassis_joint" type="fixed">
     <parent link="base_link"/>
